File: PCB/LHS Breakbeat/LHS Breakbeat.kicad_sch (KiCad schematic)
At the start: 47 parts, among them J1 Steppers In, J10 RGB, J11 Filament Sensor / Tach, J12 Endstop X, J13 Endstop Y, J14 Fan Aux, J15 Fan Part, J16 Fan Hotend/Can HL, J17 Motor X, J19 Motor X1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

Commit message: Updating BOM information
Parts:
- J1: PAIR https://eu.mouser.com/ProductDetail/Molex/43030-0001-Cut-St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 -> https://eu.mouser.com/ProductDetail/Molex/43025-2400?qs=MGl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
- J10: MFR (none) -> B3B-XH-A; PAIR (none) -> https://www.digikey.com/en/products/detail/jst-sales-americ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; URL (none) -> https://www.digikey.com/en/products/detail/jst-sales-americ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
- J11, J12, J13, J15, J16, J25, J26, J7, J8, J9: MFR (none) -> B2B-XH-A; PAIR (none) -> https://www.digikey.com/en/products/detail/jst-sales-americ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; URL (none) -> https://www.digikey.com/en/products/detail/jst-sales-americ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
- J14, J17, J19, J20, J21, J22, J23, J24: MFR (none) -> B4B-XH-A; PAIR (none) -> https://www.digikey.com/en/products/detail/jst-sales-americ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; URL (none) -> https://www.digikey.com/en/products/detail/jst-sales-americ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
- J2: PAIR https://eu.mouser.com/ProductDetail/Molex/43030-0001-Cut-St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 -> https://eu.mouser.com/ProductDetail/Molex/43025-2200?qs=KC2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
- J27: PAIR (none) -> https://eu.mouser.com/ProductDetail/Molex/50-57-9303?qs=pAY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; PAIR CRIMP (none) -> https://eu.mouser.com/ProductDetail/Molex/70058-1096?qs=gZX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
- J3: PAIR https://eu.mouser.com/ProductDetail/Molex/39-00-0208?qs=GEJ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 -> https://eu.mouser.com/ProductDetail/Molex/03-04-4052?qs=Zl0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; PAIR CRIMP https://eu.mouser.com/ProductDetail/Molex/39-00-0078?qs=53i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 -> https://eu.mouser.com/ProductDetail/Molex/45750-3112?qs=c7k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
- JP1: MFR (none) -> 22-28-5026; PAIR (none) -> https://eu.mouser.com/ProductDetail/Preci-dip/999-19-310-06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; URL (none) -> https://eu.mouser.com/ProductDetail/Molex/22-28-5026?qs=l%2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

Commit message: BOM updates, including LCSC parts, minor layout tweaks
Parts:
- D1, D2: LCSC (none) -> C2297
- D3: LCSC (none) -> C130415
- F1, F2: LCSC (none) -> C3206956; MFR Keystone 3569 -> Keystone 3568
- J1: LCSC (none) -> C277384
- J10: LCSC (none) -> C492457
- J11, J12, J13, J15, J16, J25, J26, J7, J8, J9: LCSC (none) -> C5258883
- J14, J17, J19, J20, J21, J22, J23, J24: LCSC (none) -> C709375
- J2: LCSC (none) -> C127339
- J27: LCSC (none) -> C2935911; MFR Molex 22-28-5060 -> Molex 22-28-5050; URL https://eu.mouser.com/ProductDetail/Molex/22-28-5060?qs=l%2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 -> https://eu.mouser.com/ProductDetail/Molex/22-28-5050?qs=l%2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
- J3: LCSC (none) -> C492364
- J4: LCSC (none) -> C2913282
- J5: LCSC (none) -> C428722
- JP1: LCSC (none) -> C2685195
- R1, R2: LCSC (none) -> C17673
Changed lines of the file:
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@@
+      (effects (font (size 1.27 1.27)) hide)
+    )
+    (property "LCSC" "C709375" (at 208.28 149.86 0)
       (effects (font (size 1.27 1.27)) hide)
     )
@@
       (effects (font (size 1.27 1.27)) hide)
     )
+    (property "LCSC" "C709375" (at 182.88 149.86 0)
+      (effects (font (size 1.27 1.27)) hide)
+    )
     (pin "1")
     (pin "2")
@@
     )
     (property "WIRE" "24AWG" (at 49.53 49.53 0)
+      (effects (font (size 1.27 1.27)) hide)
+    )
+    (property "LCSC" "C277384" (at 49.53 49.53 0)
       (effects (font (size 1.27 1.27)) hide)
     )
@@
       (effects (font (size 1.524 1.524)) (justify left) hide)
     )
-    (property "MFR" "Keystone 3569" (at 43.18 139.7 0)
+    (property "MFR" "Keystone 3568" (at 43.18 139.7 0)
       (effects (font (size 1.27 1.27)))
     )
@@
       (effects (font (size 1.27 1.27)) hide)
     )
+    (property "LCSC" "C3206956" (at 45.72 133.35 0)
+      (effects (font (size 1.27 1.27)) hide)
+    )
     (pin "1")
     (pin "2")
@@
     )
     (property "URL" "https://www.digikey.com/en/products/detail/jst-sales-america-inc/b2b-xh-a/1651045" (at 189.23 92.71 0)
+      (effects (font (size 1.27 1.27)) hide)
+    )
+    (property "LCSC" "C5258883" (at 189.23 92.71 0)
       (effects (font (size 1.27 1.27)) hide)
     )
@@
       (effects (font (size 1.27 1.27)) hide)
     )
+    (property "LCSC" "C2297" (at 58.42 142.24 0)
+      (effects (font (size 1.27 1.27)) hide)
+    )
     (pin "1")
     (pin "2")
@@
     )
     (property "WIRE" "24AWG" (at 105.41 48.26 0)
+      (effects (font (size 1.27 1.27)) hide)
+    )
+    (property "LCSC" "C127339" (at 105.41 48.26 0)
       (effects (font (size 1.27 1.27)) hide)
     )
@@
       (effects (font (size 1.27 1.27)) hide)
     )
+    (property "LCSC" "C709375" (at 260.35 137.16 0)
+      (effects (font (size 1.27 1.27)) hide)
+    )
     (pin "1")
     (pin "2")
@@
       (effects (font (size 1.27 1.27)) hide)
     )
+    (property "LCSC" "C2297" (at 57.15 165.1 0)
+      (effects (font (size 1.27 1.27)) hide)
+    )
     (pin "1")
     (pin "2")
@@
       (effects (font (size 1.27 1.27)) hide)
     )
+    (property "LCSC" "C709375" (at 208.28 137.16 0)
+      (effects (font (size 1.27 1.27)) hide)
+    )
     (pin "1")
     (pin "2")
@@
       (effects (font (size 1.27 1.27)) hide)
     )
+    (property "LCSC" "C709375" (at 234.95 137.16 0)
+      (effects (font (size 1.27 1.27)) hide)
+    )
     (pin "1")
     (pin "2")
@@
     )
     (property "WIRE" "16AWG" (at 54.61 92.71 0)
+      (effects (font (size 1.27 1.27)) hide)
+    )
+    (property "LCSC" "C492364" (at 54.61 92.71 0)
       (effects (font (size 1.27 1.27)) hide)
     )
@@
       (effects (font (size 1.27 1.27)) hide)
     )
+    (property "LCSC" "C130415" (at 87.63 53.34 0)
+      (effects (font (size 1.27 1.27)) hide)
+    )
     (pin "1")
     (pin "2")
@@
       (effects (font (size 1.27 1.27)) hide)
     )
+    (property "LCSC" "C2913282" (at 78.74 135.89 0)
+      (effects (font (size 1.27 1.27)) hide)
+    )
     (pin "1")
     (pin "2")
@@
       (effects (font (size 1.27 1.27)) hide)
     )
+    (property "LCSC" "C709375" (at 234.95 149.86 0)
+      (effects (font (size 1.27 1.27)) hide)
+    )
     (pin "1")
     (pin "2")
@@
     )
     (property "WIRE" "16 AWG" (at 78.74 156.21 0)
+      (effects (font (size 1.27 1.27)) hide)
+    )
+    (property "LCSC" "C428722" (at 78.74 156.21 0)
       (effects (font (size 1.27 1.27)) hide)
     )
@@
       (effects (font (size 1.27 1.27)) hide)
     )
+    (property "LCSC" "C17673" (at 64.77 165.1 0)
+      (effects (font (size 1.27 1.27)) hide)
+    )
     (pin "1")
     (pin "2")
@@
       (effects (font (size 1.27 1.27)) hide)
     )
+    (property "LCSC" "C5258883" (at 243.84 77.47 0)
+      (effects (font (size 1.27 1.27)) hide)
+    )
     (pin "1")
     (pin "2")
@@
     )
     (property "WIRE" "" (at 189.23 100.33 0)
+      (effects (font (size 1.27 1.27)) hide)
+    )
+    (property "LCSC" "C5258883" (at 189.23 100.33 0)
       (effects (font (size 1.27 1.27)) hide)
     )
@@
       (effects (font (size 1.27 1.27)) hide)
     )
+    (property "LCSC" "C5258883" (at 189.23 77.47 0)
+      (effects (font (size 1.27 1.27)) hide)
+    )
     (pin "1")
     (pin "2")
@@
       (effects (font (size 1.524 1.524)) (justify left) hide)
     )
-    (property "MFR" "Keystone 3569" (at 41.91 162.56 0)
+    (property "MFR" "Keystone 3568" (at 41.91 162.56 0)
       (effects (font (size 1.27 1.27)))
     )
@@
     )
     (property "WIRE" "" (at 44.45 156.21 0)
+      (effects (font (size 1.27 1.27)) hide)
+    )
+    (property "LCSC" "C3206956" (at 44.45 156.21 0)
       (effects (font (size 1.27 1.27)) hide)
     )
@@
       (effects (font (size 1.27 1.27)) hide)
     )
+    (property "LCSC" "C5258883" (at 180.34 38.1 0)
+      (effects (font (size 1.27 1.27)) hide)
+    )
     (pin "1")
     (pin "2")
@@
       (effects (font (size 1.27 1.27)) hide)
     )
+    (property "LCSC" "C5258883" (at 243.84 87.63 0)
+      (effects (font (size 1.27 1.27)) hide)
+    )
     (pin "1")
     (pin "2")
@@
     )
     (property "URL" "https://www.digikey.com/en/products/detail/jst-sales-america-inc/b2b-xh-a/1651045" (at 189.23 114.3 0)
+      (effects (font (size 1.27 1.27)) hide)
+    )
+    (property "LCSC" "C5258883" (at 189.23 114.3 0)
       (effects (font (size 1.27 1.27)) hide)
     )
@@
       (effects (font (size 1.27 1.27)) hide)
     )
+    (property "LCSC" "C17673" (at 66.04 142.24 0)
+      (effects (font (size 1.27 1.27)) hide)
+    )
     (pin "1")
     (pin "2")
@@
       (effects (font (size 1.27 1.27)) hide)
     )
+    (property "LCSC" "C709375" (at 243.84 99.06 0)
+      (effects (font (size 1.27 1.27)) hide)
+    )
     (pin "1")
     (pin "2")
@@
     )
     (property "URL" "https://www.digikey.com/en/products/detail/jst-sales-america-inc/B4B-XH-A/1651047" (at 182.88 137.16 0)
+      (effects (font (size 1.27 1.27)) hide)
+    )
+    (property "LCSC" "C709375" (at 182.88 137.16 0)
       (effects (font (size 1.27 1.27)) hide)
     )
@@
       (effects (font (size 1.27 1.27)) hide)
     )
+    (property "LCSC" "C5258883" (at 180.34 46.99 0)
+      (effects (font (size 1.27 1.27)) hide)
+    )
     (pin "1")
     (pin "2")
@@
       (effects (font (size 1.27 1.27)) hide)
     )
+    (property "LCSC" "C492457" (at 243.84 35.56 0)
+      (effects (font (size 1.27 1.27)) hide)
+    )
     (pin "1")
     (pin "2")
@@
     )
     (property "URL" "https://www.digikey.com/en/products/detail/jst-sales-america-inc/b2b-xh-a/1651045" (at 189.23 85.09 0)
+      (effects (font (size 1.27 1.27)) hide)
+    )
+    (property "LCSC" "C5258883" (at 189.23 85.09 0)
       (effects (font (size 1.27 1.27)) hide)
     )
@@
     )
     (property "MFR" "22-28-5026" (at 104.14 91.44 0)
-      (effects (font (size 1.27 1.27)))
+      (effects (font (size 1.27 1.27)) hide)
     )
     (property "URL" "https://eu.mouser.com/ProductDetail/Molex/22-28-5026?qs=l%252BWx29wYPrxTx4uny9SNSg%3D%3D" (at 104.14 91.44 0)
@@
       (effects (font (size 1.27 1.27)) hide)
     )
+    (property "LCSC" "C2685195" (at 104.14 91.44 0)
+      (effects (font (size 1.27 1.27)) hide)
+    )
     (pin "1")
     (pin "2")
@@
     )
     (property "URL" "https://www.digikey.com/en/products/detail/jst-sales-america-inc/b2b-xh-a/1651045" (at 180.34 54.61 0)
+      (effects (font (size 1.27 1.27)) hide)
+    )
+    (property "LCSC" "C5258883" (at 180.34 54.61 0)
       (effects (font (size 1.27 1.27)) hide)
     )
@@
       (effects (font (size 1.27 1.27)) hide)
     )
-    (property "MFR" "Molex 22-28-5060" (at 243.84 64.77 0)
-      (effects (font (size 1.27 1.27)))
-    )
-    (property "URL" "https://eu.mouser.com/ProductDetail/Molex/22-28-5060?qs=l%252BWx29wYPrz6j3%252BO38XvSA%3D%3D" (at 243.84 55.88 0)
+    (property "MFR" "Molex 22-28-5050" (at 243.84 64.77 0)
+      (effects (font (size 1.27 1.27)))
+    )
+    (property "URL" "https://eu.mouser.com/ProductDetail/Molex/22-28-5050?qs=l%252BWx29wYPryY4qe%252BU70%2FHQ%3D%3D" (at 243.84 55.88 0)
       (effects (font (size 1.27 1.27)) hide)
     )
@@
       (effects (font (size 1.27 1.27)) hide)
     )
+    (property "LCSC" "C2935911" (at 243.84 55.88 0)
+      (effects (font (size 1.27 1.27)) hide)
+    )

Commit message: Acknowledgements and small BOM tweaks.
Parts:
- D2: MFR (none) -> HSMG-C170
Changed lines of the file:
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@@
       (effects (font (size 1.27 1.27)) hide)
     )
-    (property "MFR" "" (at 57.15 165.1 0)
-      (effects (font (size 1.27 1.27)))
+    (property "MFR" "HSMG-C170" (at 57.15 165.1 0)
+      (effects (font (size 1.27 1.27)) hide)
     )
     (property "URL" "https://www.tme.eu/is/en/details/hsmg-c170/smd-colour-leds/broadcom-avago/" (at 57.15 165.1 0)

Commit message: Adding LHS Breakbeat Wiring Harness specifications
Parts:
- F1: PAIR (none) -> Fuse Mini 297 10A
- F2: PAIR (none) -> Fuse Mini 297 5A
- J3: LCSC C492364 -> C485326
- J4: symbol Connector_Generic:Conn_01x04 -> Connector_Generic:Conn_01x02
Changed lines of the file:
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@@
-    (stroke (width 0) (type default))
-  )
-  (wire (pts (xy 73.66 135.89) (xy 69.85 135.89))
     (stroke (width 0) (type default))
   )
@@
     (stroke (width 0) (type default))
   )
+  (wire (pts (xy 69.85 135.89) (xy 73.66 135.89))
+    (stroke (width 0) (type default))
+  )
   (wire (pts (xy 237.49 60.96) (xy 240.03 60.96))
     (stroke (width 0) (type default))
@@
     (effects (font (size 1.27 1.27)) (justify left bottom))
   )
-  (text "Endstops\n" (at 167.64 72.39 0)
+  (text "Endstops" (at 167.64 72.39 0)
     (effects (font (size 1.27 1.27)) (justify left bottom))
   )
@@
     (effects (font (size 1.27 1.27)) (justify left bottom))
   )
-  (text "Ports\n" (at 146.05 19.05 0)
+  (text "Ports" (at 146.05 19.05 0)
     (effects (font (size 1.27 1.27) (thickness 0.254) bold) (justify left bottom))
   )
@@
     (effects (font (size 1.27 1.27)) (justify left bottom))
   )
-  (text "RGB\n" (at 223.52 29.21 0)
+  (text "RGB" (at 223.52 29.21 0)
     (effects (font (size 1.27 1.27)) (justify left bottom))
   )
@@
       (effects (font (size 1.27 1.27)) hide)
     )
-    (property "PAIR" "" (at 45.72 133.35 0)
+    (property "PAIR" "Fuse Mini 297 10A" (at 45.72 133.35 0)
       (effects (font (size 1.27 1.27)) hide)
     )
@@
       (effects (font (size 1.27 1.27)) hide)
     )
-    (property "LCSC" "C492364" (at 54.61 92.71 0)
+    (property "LCSC" "C485326" (at 54.61 92.71 0)
       (effects (font (size 1.27 1.27)) hide)
     )
@@
     )
   )
-  (symbol (lib_id "Connector_Generic:Conn_01x04") (at 78.74 135.89 0) (unit 1)
-    (in_bom yes) (on_board yes) (dnp no)
-    (property "Reference" "J4" (at 81.28 137.16 0)
-      (effects (font (size 1.27 1.27)) (justify left))
-    )
-    (property "Value" "Hotend / Can 24V" (at 71.12 144.78 0)
-      (effects (font (size 1.27 1.27)) (justify left))
-    )
-    (property "Footprint" "Mouser:XT30PWF" (at 78.74 135.89 0)
-      (effects (font (size 1.27 1.27)) hide)
-    )
-    (property "Datasheet" "~" (at 78.74 135.89 0)
-      (effects (font (size 1.27 1.27)) hide)
-    )
-    (property "MFR" "Amass XT30PW-F" (at 78.74 148.59 0)
-      (effects (font (size 1.27 1.27)))
-    )
-    (property "URL" "https://www.tme.eu/is/en/details/xt30pw-f/dc-power-connectors/amass/?utm_campaign=stock-2024-02-03&utm_medium=cpc&utm_source=findchips.com" (at 78.74 135.89 0)
-      (effects (font (size 1.27 1.27)) hide)
-    )
-    (property "CRIMP" "" (at 78.74 135.89 0)
-      (effects (font (size 1.27 1.27)) hide)
-    )
-    (property "PAIR" "https://www.tme.eu/is/en/details/xt30u-m/dc-power-connectors/amass/" (at 78.74 135.89 0)
-      (effects (font (size 1.27 1.27)) hide)
-    )
-    (property "PAIR CRIMP" "" (at 78.74 135.89 0)
-      (effects (font (size 1.27 1.27)) hide)
-    )
-    (property "WIRE" "18 AWG" (at 78.74 135.89 0)
-      (effects (font (size 1.27 1.27)) hide)
-    )
-    (property "LCSC" "C2913282" (at 78.74 135.89 0)
+  (symbol (lib_id "Connector_Generic:Conn_01x02") (at 78.74 133.35 0) (unit 1)
+    (in_bom yes) (on_board yes) (dnp no)
+    (property "Reference" "J4" (at 81.28 134.62 0)
+      (effects (font (size 1.27 1.27)) (justify left))
+    )
+    (property "Value" "Hotend / Can 24V" (at 71.12 142.24 0)
+      (effects (font (size 1.27 1.27)) (justify left))
+    )
+    (property "Footprint" "Mouser:XT30PWF" (at 78.74 133.35 0)
+      (effects (font (size 1.27 1.27)) hide)
+    )
+    (property "Datasheet" "~" (at 78.74 133.35 0)
+      (effects (font (size 1.27 1.27)) hide)
+    )
+    (property "MFR" "Amass XT30PW-F" (at 78.74 146.05 0)
+      (effects (font (size 1.27 1.27)))
+    )
+    (property "URL" "https://www.tme.eu/is/en/details/xt30pw-f/dc-power-connectors/amass/?utm_campaign=stock-2024-02-03&utm_medium=cpc&utm_source=findchips.com" (at 78.74 133.35 0)
+      (effects (font (size 1.27 1.27)) hide)
+    )
+    (property "CRIMP" "" (at 78.74 133.35 0)
+      (effects (font (size 1.27 1.27)) hide)
+    )
+    (property "PAIR" "https://www.tme.eu/is/en/details/xt30u-m/dc-power-connectors/amass/" (at 78.74 133.35 0)
+      (effects (font (size 1.27 1.27)) hide)
+    )
+    (property "PAIR CRIMP" "" (at 78.74 133.35 0)
+      (effects (font (size 1.27 1.27)) hide)
+    )
+    (property "WIRE" "18 AWG" (at 78.74 133.35 0)
+      (effects (font (size 1.27 1.27)) hide)
+    )
+    (property "LCSC" "C2913282" (at 78.74 133.35 0)
+      (effects (font (size 1.27 1.27)) hide)
+    )
+    (pin "1")
+    (pin "2")
+    (instances
+      (project "LHS Breakbeat"
+        (path "/bba6e55c-03b8-4eb9-ac5d-8eef535ad508"
+          (reference "J4") (unit 1)
+        )
+      )
+    )
+  )
+  (symbol (lib_id "Mechanical:Fiducial") (at 137.16 190.5 0) (unit 1)
+    (in_bom no) (on_board yes) (dnp no)
+    (property "Reference" "FID3" (at 139.319 189.3316 0)
+      (effects (font (size 1.27 1.27)) (justify left))
+    )
+    (property "Value" "Fiducial" (at 139.319 191.643 0)
+      (effects (font (size 1.27 1.27)) (justify left))
+    )
+    (property "Footprint" "Fiducial:Fiducial_1.5mm_Mask3mm" (at 137.16 190.5 0)
+      (effects (font (size 1.27 1.27)) hide)
+    )
+    (property "Datasheet" "~" (at 137.16 190.5 0)
+      (effects (font (size 1.27 1.27)) hide)
+    )
+    (instances
+      (project "LHS Breakbeat"
+        (path "/bba6e55c-03b8-4eb9-ac5d-8eef535ad508"
+          (reference "FID3") (unit 1)
+        )
+      )
+      (project "Leviathan"
+        (path "/d0de4886-c3c5-428d-a439-eb59fb6f1a43"
+          (reference "FID3") (unit 1)
+        )
+      )
+    )
+  )
+  (symbol (lib_id "Connector_Generic:Conn_01x04") (at 234.95 149.86 0) (unit 1)
+    (in_bom yes) (on_board yes) (dnp no)
+    (property "Reference" "J21" (at 237.49 149.86 0)
+      (effects (font (size 1.27 1.27)) (justify left))
+    )
+    (property "Value" "Motor Z1" (at 237.49 152.4 0)
+      (effects (font (size 1.27 1.27)) (justify left))
+    )
+    (property "Footprint" "Connector_JST:JST_XH_B4B-XH-A_1x04_P2.50mm_Vertical" (at 234.95 149.86 0)
+      (effects (font (size 1.27 1.27)) hide)
+    )
+    (property "Datasheet" "~" (at 234.95 149.86 0)
+      (effects (font (size 1.27 1.27)) hide)
+    )
+    (property "MFR" "B4B-XH-A" (at 234.95 149.86 0)
+      (effects (font (size 1.27 1.27)) hide)
+    )
+    (property "PAIR" "https://www.digikey.com/en/products/detail/jst-sales-america-inc/XHP-4/683353" (at 234.95 149.86 0)
+      (effects (font (size 1.27 1.27)) hide)
+    )
+    (property "URL" "https://www.digikey.com/en/products/detail/jst-sales-america-inc/B4B-XH-A/1651047" (at 234.95 149.86 0)
+      (effects (font (size 1.27 1.27)) hide)
+    )
+    (property "LCSC" "C709375" (at 234.95 149.86 0)
       (effects (font (size 1.27 1.27)) hide)
     )
@@
       (project "LHS Breakbeat"
         (path "/bba6e55c-03b8-4eb9-ac5d-8eef535ad508"
-          (reference "J4") (unit 1)
-        )
-      )
-    )
-  )
-  (symbol (lib_id "Mechanical:Fiducial") (at 137.16 190.5 0) (unit 1)
-    (in_bom no) (on_board yes) (dnp no)
-    (property "Reference" "FID3" (at 139.319 189.3316 0)
-      (effects (font (size 1.27 1.27)) (justify left))
-    )
-    (property "Value" "Fiducial" (at 139.319 191.643 0)
-      (effects (font (size 1.27 1.27)) (justify left))
-    )
-    (property "Footprint" "Fiducial:Fiducial_1.5mm_Mask3mm" (at 137.16 190.5 0)
-      (effects (font (size 1.27 1.27)) hide)
-    )
-    (property "Datasheet" "~" (at 137.16 190.5 0)
-      (effects (font (size 1.27 1.27)) hide)
-    )
-    (instances
-      (project "LHS Breakbeat"
-        (path "/bba6e55c-03b8-4eb9-ac5d-8eef535ad508"
-          (reference "FID3") (unit 1)
-        )
-      )
-      (project "Leviathan"
-        (path "/d0de4886-c3c5-428d-a439-eb59fb6f1a43"
-          (reference "FID3") (unit 1)
-        )
-      )
-    )
-  )
-  (symbol (lib_id "Connector_Generic:Conn_01x04") (at 234.95 149.86 0) (unit 1)
-    (in_bom yes) (on_board yes) (dnp no)
-    (property "Reference" "J21" (at 237.49 149.86 0)
-      (effects (font (size 1.27 1.27)) (justify left))
-    )
-    (property "Value" "Motor Z1" (at 237.49 152.4 0)
-      (effects (font (size 1.27 1.27)) (justify left))
-    )
-    (property "Footprint" "Connector_JST:JST_XH_B4B-XH-A_1x04_P2.50mm_Vertical" (at 234.95 149.86 0)
-      (effects (font (size 1.27 1.27)) hide)
-    )
-    (property "Datasheet" "~" (at 234.95 149.86 0)
-      (effects (font (size 1.27 1.27)) hide)
-    )
-    (property "MFR" "B4B-XH-A" (at 234.95 149.86 0)
-      (effects (font (size 1.27 1.27)) hide)
-    )
-    (property "PAIR" "https://www.digikey.com/en/products/detail/jst-sales-america-inc/XHP-4/683353" (at 234.95 149.86 0)
-      (effects (font (size 1.27 1.27)) hide)
-    )
-    (property "URL" "https://www.digikey.com/en/products/detail/jst-sales-america-inc/B4B-XH-A/1651047" (at 234.95 149.86 0)
-      (effects (font (size 1.27 1.27)) hide)
-    )
-    (property "LCSC" "C709375" (at 234.95 149.86 0)
-      (effects (font (size 1.27 1.27)) hide)
-    )
-    (pin "1")
-    (pin "2")
-    (pin "3")
-    (pin "4")
-    (instances
-      (project "LHS Breakbeat"
-        (path "/bba6e55c-03b8-4eb9-ac5d-8eef535ad508"
           (reference "J21") (unit 1)
         )
@@
       (effects (font (size 1.27 1.27)) hide)
     )
-    (property "PAIR" "" (at 44.45 156.21 0)
-      (effects (font (size 1.27 1.27)) hide)
-    )
+    (property "PAIR" "Fuse Mini 297 5A" (at 44.45 156.21 0)
+      (effects (font (size 1.27 1.27)) hide)
+    )
