File: PCB/PI Bed Heater - 200mm/KiCad/HeatedBedFoil.kicad_pcb (KiCad board)
At the start: 2 copper layers, 200 x 200 mm, 2 parts, among them J1 Screw_Terminal_01x01

Commit message: updated heatbed instructions
Parts:
- J1: value Screw_Terminal_01x01 -> Pad
- J2: renamed from J1; value Screw_Terminal_01x01 -> Pad
Changed lines of the file:
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@@
         (effects (font (size 1 1) (thickness 0.15)))
     )
-    (fp_text value "Screw_Terminal_01x01" (at 1 10 90) (layer "F.Fab") hide
+    (fp_text value "Pad" (at 1 10 90) (layer "F.Fab") hide
         (effects (font (size 1 1) (thickness 0.15)))
     )
@@
     (tags "test point SMD pad rectangle square")
     (attr exclude_from_pos_files exclude_from_bom)
-    (fp_text reference "J1" (at 0 -2.898 90) (layer "F.SilkS") hide
+    (fp_text reference "J2" (at 0 -2.898 90) (layer "F.SilkS") hide
         (effects (font (size 1 1) (thickness 0.15)))
     )
-    (fp_text value "Screw_Terminal_01x01" (at 1 10 90) (layer "F.Fab") hide
+    (fp_text value "Pad" (at 1 10 90) (layer "F.Fab") hide
         (effects (font (size 1 1) (thickness 0.15)))
     )
