File: PCB/PI Bed Heater - 200mm/KiCad/HeatedBedFoil.kicad_sch (KiCad schematic)
At the start: 0 parts

Commit message: updated heatbed instructions
Parts:
- added TP1: +24V, symbol Connector:TestPoint
- added TP2: GND, symbol Connector:TestPoint
Connections:
- new net: TP1.1, TP2.1
Changed lines of the file:
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@@
 (kicad_sch (version 20230121) (generator eeschema)
   (paper "A4")
+  (wire (pts (xy 138.43 95.25) (xy 143.51 95.25))
+    (stroke (width 0) (type default))
+  )
+  (wire (pts (xy 153.67 90.17) (xy 158.75 90.17))
+    (stroke (width 0) (type default))
+  )
+  (wire (pts (xy 148.59 90.17) (xy 148.59 95.25))
+    (stroke (width 0) (type default))
+  )
+  (wire (pts (xy 148.59 95.25) (xy 153.67 95.25))
+    (stroke (width 0) (type default))
+  )
+  (wire (pts (xy 153.67 95.25) (xy 153.67 90.17))
+    (stroke (width 0) (type default))
+  )
+  (wire (pts (xy 143.51 90.17) (xy 148.59 90.17))
+    (stroke (width 0) (type default))
+  )
+  (wire (pts (xy 138.43 90.17) (xy 138.43 95.25))
+    (stroke (width 0) (type default))
+  )
+  (wire (pts (xy 143.51 95.25) (xy 143.51 90.17))
+    (stroke (width 0) (type default))
+  )
+  (wire (pts (xy 133.35 90.17) (xy 138.43 90.17))
+    (stroke (width 0) (type default))
+  )
+  (symbol (lib_id "Connector:TestPoint") (at 133.35 90.17 0) (unit 1)
+    (in_bom yes) (on_board yes) (dnp no) (fields_autoplaced)
+    (property "Reference" "TP1" (at 135.89 85.598 0)
+      (effects (font (size 1.27 1.27)) (justify left))
+    )
+    (property "Value" "+24V" (at 135.89 88.138 0)
+      (effects (font (size 1.27 1.27)) (justify left))
+    )
+    (property "Footprint" "" (at 138.43 90.17 0)
+      (effects (font (size 1.27 1.27)) hide)
+    )
+    (property "Datasheet" "~" (at 138.43 90.17 0)
+      (effects (font (size 1.27 1.27)) hide)
+    )
+    (pin "1")
+    (instances
+      (project "HeatedBedFoil"
+        (path "/0b27d95d-56a4-4b2a-b388-4b89902e9c5e"
+          (reference "TP1") (unit 1)
+        )
+      )
+    )
+  )
+  (symbol (lib_id "Connector:TestPoint") (at 158.75 90.17 0) (unit 1)
+    (in_bom yes) (on_board yes) (dnp no) (fields_autoplaced)
+    (property "Reference" "TP2" (at 161.29 85.598 0)
+      (effects (font (size 1.27 1.27)) (justify left))
+    )
+    (property "Value" "GND" (at 161.29 88.138 0)
+      (effects (font (size 1.27 1.27)) (justify left))
+    )
+    (property "Footprint" "" (at 163.83 90.17 0)
+      (effects (font (size 1.27 1.27)) hide)
+    )
+    (property "Datasheet" "~" (at 163.83 90.17 0)
+      (effects (font (size 1.27 1.27)) hide)
+    )
+    (pin "1")
+    (instances
+      (project "HeatedBedFoil"
+        (path "/0b27d95d-56a4-4b2a-b388-4b89902e9c5e"
+          (reference "TP2") (unit 1)
+        )
+      )
+    )
+  )
   (sheet_instances
     (path "/" (page "1"))
