File: User_Mods/Printer/Y Tensioner PCB Retainer Plate - @LH/KiCad/Y Tensioner Plate.kicad_pcb (KiCad board)
At the start: 2 copper layers, 53 x 27 mm, 2 parts

Commit message: updating ordering instructions
Other:
- board text added: "JLCJLCJLC"
Changed lines of the file:
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@@
   (gr_line (start 179.580566 87.347581) (end 179.489395 87.26902)
     (stroke (width 0.224375) (type solid)) (layer "Edge.Cuts"))
+  (gr_text "JLCJLCJLC" (at 173.675977 112.662591) (layer "B.SilkS")
+    (effects (font (size 0.8 0.8) (thickness 0.1)) (justify left bottom mirror))
+  )
   (dimension (type aligned) (layer "Dwgs.User")
     (pts (xy 135 114) (xy 135 87))
